File: KosmoTuringJack/TuringJack.kicad_pcb (KiCad board)
At the start: 2 copper layers, 95 x 50 mm, 10 parts, among them J1 Conn_01x10_Female

Commit message: fix #1 missing cathode connection of clock led
Connections:
- CLK1 pad 1: unconnected-(CLK1-Pad1) -> /GND
Changed lines of the file:
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@@
   (net 8 "unconnected-(J1-Pad9)")
   (net 9 "Net-(PULS1-Pad2)")
-  (net 10 "unconnected-(CLK1-Pad1)")
-  (net 11 "Net-(CLK1-Pad2)")
-  (net 12 "/CLOCK_J")
+  (net 10 "Net-(CLK1-Pad2)")
+  (net 11 "/CLOCK_J")
   (footprint "ao_tht:Jack_6.35mm_PJ_629HAN" (layer "F.Cu")
     (at 37.5 200 -90)
@@
       (net 1 "/GND") (pinfunction "Pin_1") (pintype "passive"))
     (pad "2" thru_hole oval (at 0 2.54 90) (size 1.7 1.7) (drill 1) (layers *.Cu *.Mask)
-      (net 12 "/CLOCK_J") (pinfunction "Pin_2") (pintype "passive"))
+      (net 11 "/CLOCK_J") (pinfunction "Pin_2") (pintype "passive"))
     (pad "3" thru_hole oval (at 0 5.08 90) (size 1.7 1.7) (drill 1) (layers *.Cu *.Mask)
       (net 2 "/CLOCK_IN_J") (pinfunction "Pin_3") (pintype "passive"))
@@
     (fp_line (start 1.93 1.25) (end 8.23 1.25) (layer "F.Fab") (width 0.1))
     (pad "1" thru_hole circle locked (at 0 0 270) (size 1.6 1.6) (drill 0.8) (layers *.Cu *.Mask)
-      (net 12 "/CLOCK_J") (pintype "passive"))
+      (net 11 "/CLOCK_J") (pintype "passive"))
     (pad "2" thru_hole oval locked (at 10.16 0 270) (size 1.6 1.6) (drill 0.8) (layers *.Cu *.Mask)
-      (net 11 "Net-(CLK1-Pad2)") (pintype "passive"))
+      (net 10 "Net-(CLK1-Pad2)") (pintype "passive"))
     (model "${KICAD_AOKICAD}/ao_tht_3d/R_Axial_DIN0207_L6.3mm_D2.5mm_P10.16mm_Horizontal.wrl"
       (offset (xyz 0 0 0))
@@
     (fp_circle (center 1.27 0) (end 3.77 0) (layer "F.Fab") (width 0.1) (fill none))
     (pad "1" thru_hole rect locked (at 0 0) (size 1.8 1.8) (drill 0.9) (layers *.Cu *.Mask)
-      (net 10 "unconnected-(CLK1-Pad1)") (pinfunction "K") (pintype "passive"))
+      (net 1 "/GND") (pinfunction "K") (pintype "passive"))
     (pad "2" thru_hole circle locked (at 2.54 0) (size 1.8 1.8) (drill 0.9) (layers *.Cu *.Mask)
-      (net 11 "Net-(CLK1-Pad2)") (pinfunction "A") (pintype "passive"))
+      (net 10 "Net-(CLK1-Pad2)") (pinfunction "A") (pintype "passive"))
     (model "${KICAD_AOKICAD}/ao_tht_3d/LED_D5.0mm.wrl"
       (offset (xyz 0 0 0))
@@
   (segment (start 68.834 184.15) (end 93.915 184.15) (width 0.25) (layer "F.Cu") (net 9))
   (segment (start 93.915 184.15) (end 99.265 189.5) (width 0.25) (layer "F.Cu") (net 9))
-  (segment (start 54.61 187.706) (end 52.816 189.5) (width 0.25) (layer "F.Cu") (net 11))
-  (segment (start 52.816 189.5) (end 49.265 189.5) (width 0.25) (layer "F.Cu") (net 11))
-  (segment (start 54.61 184.15) (end 54.61 187.706) (width 0.25) (layer "F.Cu") (net 11))
-  (segment (start 54.61 162.545) (end 54.61 173.99) (width 0.25) (layer "F.Cu") (net 12))
-  (segment (start 54.68 162.475) (end 54.61 162.545) (width 0.25) (layer "F.Cu") (net 12))
+  (segment (start 54.61 187.706) (end 52.816 189.5) (width 0.25) (layer "F.Cu") (net 10))
+  (segment (start 52.816 189.5) (end 49.265 189.5) (width 0.25) (layer "F.Cu") (net 10))
+  (segment (start 54.61 184.15) (end 54.61 187.706) (width 0.25) (layer "F.Cu") (net 10))
+  (segment (start 54.61 162.545) (end 54.61 173.99) (width 0.25) (layer "F.Cu") (net 11))
+  (segment (start 54.68 162.475) (end 54.61 162.545) (width 0.25) (layer "F.Cu") (net 11))
   (zone (net 1) (net_name "/GND") (layer "F.Cu") (hatch edge 0.508)
     (connect_pads (clearance 0.508))

Commit message: move pulse out 1k resistor after the led, so it does not act as voltage divider, thanks @holmesrichards !
Parts:
- added R3: 1k, ao_tht:R_Axial_DIN0207_L6.3mm_D2.5mm_P10.16mm_Horizontal, F.Cu at (73.7, 174.0)
Connections:
- PULSE_OUT1 pad T: /PULSE_OUT_J -> Net-(PULSE_OUT1-PadT)
Routing:
- net /PULSE_OUT_J: track 47.4 -> 16.9 mm
- net Net-(PULSE_OUT1-PadT): track 0.00 -> 17.3 mm
- net Net-(PULS1-Pad2): track 32.6 -> 35.4 mm
Changed lines of the file:
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@@
   (net 10 "Net-(CLK1-Pad2)")
   (net 11 "/CLOCK_J")
+  (net 12 "Net-(PULSE_OUT1-PadT)")
   (footprint "ao_tht:Jack_6.35mm_PJ_629HAN" (layer "F.Cu")
     (at 37.5 200 -90)
@@
     )
   )
+  (footprint "ao_tht:R_Axial_DIN0207_L6.3mm_D2.5mm_P10.16mm_Horizontal" (layer "F.Cu")
+    (at 73.66 173.99 -90)
+    (descr "Resistor, Axial_DIN0207 series, Axial, Horizontal, pin pitch=10.16mm, 0.25W = 1/4W, length*diameter=6.3*2.5mm^2, http://cdn-reichelt.de/documents/datenblatt/B400/1_4W%23YAG.pdf")
+    (tags "Resistor Axial_DIN0207 series Axial Horizontal pin pitch 10.16mm 0.25W = 1/4W length 6.3mm diameter 2.5mm")
+    (property "Sheetfile" "TuringJack.kicad_sch")
+    (property "Sheetname" "")
+    (property "Vendor" "Tayda")
+    (attr through_hole)
+    (fp_text reference "R3" (at 5.08 -2.37 90) (layer "F.SilkS")
+      (effects (font (size 0.75 0.75) (thickness 0.15)))
+    )
+    (fp_text value "1k" (at 5.08 2.37 90) (layer "F.Fab")
+      (effects (font (size 1 1) (thickness 0.15)))
+    )
+    (fp_text user "${VALUE}" (at 5.08 0 90) (layer "F.SilkS")
+      (effects (font (size 0.75 0.75) (thickness 0.15)))
+    )
+    (fp_text user "${REFERENCE}" (at 5.08 0 90) (layer "F.Fab")
+      (effects (font (size 1 1) (thickness 0.15)))
+    )
+    (fp_line (start 1.04 0) (end 1.81 0) (layer "F.SilkS") (width 0.12))
+    (fp_line (start 9.12 0) (end 8.35 0) (layer "F.SilkS") (width 0.12))
+    (fp_line (start 8.35 1.37) (end 8.35 -1.37) (layer "F.SilkS") (width 0.12))
+    (fp_line (start 1.81 -1.37) (end 1.81 1.37) (layer "F.SilkS") (width 0.12))
+    (fp_line (start 8.35 -1.37) (end 1.81 -1.37) (layer "F.SilkS") (width 0.12))
+    (fp_line (start 1.81 1.37) (end 8.35 1.37) (layer "F.SilkS") (width 0.12))
+    (fp_line (start -1.05 1.5) (end 11.21 1.5) (layer "F.CrtYd") (width 0.05))
+    (fp_line (start 11.21 1.5) (end 11.21 -1.5) (layer "F.CrtYd") (width 0.05))
+    (fp_line (start 11.21 -1.5) (end -1.05 -1.5) (layer "F.CrtYd") (width 0.05))
+    (fp_line (start -1.05 -1.5) (end -1.05 1.5) (layer "F.CrtYd") (width 0.05))
+    (fp_line (start 8.23 1.25) (end 8.23 -1.25) (layer "F.Fab") (width 0.1))
+    (fp_line (start 1.93 -1.25) (end 1.93 1.25) (layer "F.Fab") (width 0.1))
+    (fp_line (start 1.93 1.25) (end 8.23 1.25) (layer "F.Fab") (width 0.1))
+    (fp_line (start 0 0) (end 1.93 0) (layer "F.Fab") (width 0.1))
+    (fp_line (start 10.16 0) (end 8.23 0) (layer "F.Fab") (width 0.1))
+    (fp_line (start 8.23 -1.25) (end 1.93 -1.25) (layer "F.Fab") (width 0.1))
+    (pad "1" thru_hole circle locked (at 0 0 270) (size 1.6 1.6) (drill 0.8) (layers *.Cu *.Mask)
+      (net 6 "/PULSE_OUT_J") (pintype "passive"))
+    (pad "2" thru_hole oval locked (at 10.16 0 270) (size 1.6 1.6) (drill 0.8) (layers *.Cu *.Mask)
+      (net 12 "Net-(PULSE_OUT1-PadT)") (pintype "passive"))
+    (model "${KICAD_AOKICAD}/ao_tht_3d/R_Axial_DIN0207_L6.3mm_D2.5mm_P10.16mm_Horizontal.wrl"
+      (offset (xyz 0 0 0))
+      (scale (xyz 1 1 1))
+      (rotate (xyz 0 0 0))
+    )
+  )
   (footprint "ao_tht:Jack_6.35mm_PJ_629HAN" (layer "F.Cu")
     (at 112.5 200 -90)
@@
       (net 1 "/GND") (pintype "passive"))
     (pad "T" thru_hole circle locked (at -6.4 0.5 270) (size 4.5 4.5) (drill 2.7) (layers *.Cu *.Mask)
-      (net 6 "/PULSE_OUT_J") (pintype "passive"))
+      (net 12 "Net-(PULSE_OUT1-PadT)") (pintype "passive"))
     (pad "TN" thru_hole circle locked (at -2.5 6.4 270) (size 4.5 4.5) (drill 2.7) (layers *.Cu *.Mask))
     (model "${KICAD_USER_LIBRARY}/aoKicad/ao_tht_3d/User Library-jack-4.STEP"
@@
   (segment (start 62 165.315) (end 64.84 162.475) (width 0.25) (layer "F.Cu") (net 5))
   (segment (start 68.834 163.929) (end 68.834 173.99) (width 0.25) (layer "F.Cu") (net 6))
+  (segment (start 68.834 173.99) (end 73.66 173.99) (width 0.25) (layer "F.Cu") (net 6))
   (segment (start 67.38 162.475) (end 68.834 163.929) (width 0.25) (layer "F.Cu") (net 6))
-  (segment (start 68.834 173.99) (end 82.804 173.99) (width 0.25) (layer "B.Cu") (net 6))
-  (segment (start 87 178.186) (end 87 193.6) (width 0.25) (layer "B.Cu") (net 6))
-  (segment (start 82.804 173.99) (end 87 178.186) (width 0.25) (layer "B.Cu") (net 6))
   (segment (start 96 165) (end 112 181) (width 0.25) (layer "F.Cu") (net 7))
   (segment (start 72.445 165) (end 96 165) (width 0.25) (layer "F.Cu") (net 7))
   (segment (start 69.92 162.475) (end 72.445 165) (width 0.25) (layer "F.Cu") (net 7))
   (segment (start 112 181) (end 112 193.6) (width 0.25) (layer "F.Cu") (net 7))
-  (segment (start 68.834 184.15) (end 93.915 184.15) (width 0.25) (layer "F.Cu") (net 9))
-  (segment (start 93.915 184.15) (end 99.265 189.5) (width 0.25) (layer "F.Cu") (net 9))
+  (segment (start 72.136 180.848) (end 90.613 180.848) (width 0.25) (layer "F.Cu") (net 9))
+  (segment (start 68.834 184.15) (end 72.136 180.848) (width 0.25) (layer "F.Cu") (net 9))
+  (segment (start 90.613 180.848) (end 99.265 189.5) (width 0.25) (layer "F.Cu") (net 9))
   (segment (start 54.61 187.706) (end 52.816 189.5) (width 0.25) (layer "F.Cu") (net 10))
   (segment (start 52.816 189.5) (end 49.265 189.5) (width 0.25) (layer "F.Cu") (net 10))
@@
   (segment (start 54.61 162.545) (end 54.61 173.99) (width 0.25) (layer "F.Cu") (net 11))
   (segment (start 54.68 162.475) (end 54.61 162.545) (width 0.25) (layer "F.Cu") (net 11))
+  (segment (start 77.55 184.15) (end 87 193.6) (width 0.25) (layer "B.Cu") (net 12))
+  (segment (start 73.66 184.15) (end 77.55 184.15) (width 0.25) (layer "B.Cu") (net 12))
   (zone (net 1) (net_name "/GND") (layer "F.Cu") (hatch edge 0.508)
     (connect_pads (clearance 0.508))
