File: KosmoTuringMain/TuringMain.kicad_sch (KiCad schematic)
At the start: 106 parts, among them IC1 TL072P, IC2 78L09, IC3 78L09, J1 Conn_01x10_Female, J2 Conn_01x10_Male, T1 2N3904, U1 TL074_

Commit message: move pulse out 1k resistor after the led, so it does not act as voltage divider, thanks @holmesrichards !
Parts:
- removed R39: 1k, ao_tht:R_Axial_DIN0207_L6.3mm_D2.5mm_P10.16mm_Horizontal, symbol ao_symbols:R
Connections:
- net PULSE_OUT: now also BUFFER1.15 (O)
Changed lines of the file:
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@@
     (effects (font (size 0.7112 0.7112)) (justify right bottom))
   )
-  (label "PULSE_OUT" (at 545.465 307.975 0)
+  (label "PULSE_OUT" (at 537.845 307.975 0)
     (effects (font (size 0.7112 0.7112)) (justify left bottom))
   )
@@
     (pin "14")
   )
-  (symbol (lib_id "ao_symbols:R") (at 541.655 307.975 270) (unit 1)
-    (in_bom yes) (on_board yes)
-    (property "Reference" "R39" (id 0) (at 539.115 311.785 90)
-      (effects (font (size 1.778 1.5113)) (justify left bottom))
-    )
-    (property "Value" "1k" (id 1) (at 539.115 306.705 90)
-      (effects (font (size 1.778 1.5113)) (justify left bottom))
-    )
-    (property "Footprint" "ao_tht:R_Axial_DIN0207_L6.3mm_D2.5mm_P10.16mm_Horizontal" (id 2) (at 541.655 306.197 90)
-      (effects (font (size 1.27 1.27)) hide)
-    )
-    (property "Datasheet" "" (id 3) (at 541.655 307.975 0)
-      (effects (font (size 1.27 1.27)) hide)
-    )
-    (property "Vendor" "Tayda" (id 4) (at 541.655 307.975 0)
-      (effects (font (size 1.27 1.27)) hide)
-    )
-    (pin "1")
-    (pin "2")
-  )
   (symbol (lib_id "TuringBack-eagle-import:TL072P") (at 338.455 67.945 0) (unit 1)
     (in_bom yes) (on_board yes)
@@
       (reference "R38") (unit 1) (value "2.2k") (footprint "ao_tht:R_Axial_DIN0207_L6.3mm_D2.5mm_P10.16mm_Horizontal")
     )
-    (path "/1840c087-7e91-41f1-a09f-34fbc7881e29"
-      (reference "R39") (unit 1) (value "1k") (footprint "ao_tht:R_Axial_DIN0207_L6.3mm_D2.5mm_P10.16mm_Horizontal")
-    )
     (path "/cc2ebcc1-7b9a-4332-97f0-fe8dd2d9bd70"
